File: Batterietester.kicad_pcb (KiCad board)
At the start: 2 copper layers, 67 x 53 mm, 22 parts, among them J1 Screw_Terminal_1x02, J2 Screw_Terminal_1x02, J3 Screw_Terminal_1x02, J4 CONN_01X02, SW1 SW_Push, SW2 SW_Push, U1 LM3914

Commit message: cleaning
Changed lines of the file:
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@@
     (links 52)
     (no_connects 0)
-    (area 80.575001 60.125 180.275 132.525001)
+    (area 98.349999 70.749999 165.500001 123.900001)
     (thickness 1.6)
     (drawings 35)
@@
       (effects (font (size 1 1) (thickness 0.15)))
     )
-    (fp_text value LM3914 (at 3.81 22.65 180) (layer F.Fab)
+    (fp_text value LM3914 (at 3.81 22.65 180) (layer F.SilkS)
       (effects (font (size 1 1) (thickness 0.15)))
     )
@@
       (effects (font (size 1 1) (thickness 0.15)))
     )
-    (fp_text value 10k (at 5.08 2.31) (layer F.Fab)
+    (fp_text value 10k (at 5.1 2.14) (layer F.SilkS)
       (effects (font (size 1 1) (thickness 0.15)))
     )
@@
       (effects (font (size 1 1) (thickness 0.15)))
     )
-    (fp_text value 20k (at 5.08 2.31) (layer F.Fab)
+    (fp_text value 20k (at 5.08 -1.905) (layer F.SilkS)
       (effects (font (size 1 1) (thickness 0.15)))
     )
@@
     (descr "single turn cermet trimmer, Copal CT-6EP, https://www.nidec-copal-electronics.com/e/catalog/trimmer/ct-6.pdf")
     (tags "potentiometer trimmer")
-    (fp_text reference RV1 (at 0 -2) (layer F.SilkS)
-      (effects (font (size 1 1) (thickness 0.15)))
-    )
-    (fp_text value 10k (at 0 7) (layer F.Fab)
+    (fp_text reference RV1 (at 0 2.54) (layer F.SilkS)
+      (effects (font (size 1 1) (thickness 0.15)))
+    )
+    (fp_text value 10k (at 5.08 3.81) (layer F.SilkS)
       (effects (font (size 1 1) (thickness 0.15)))
     )
@@
     (descr https://www.omron.com/ecb/products/pdf/en-b3f.pdf)
     (tags "tact sw push 6mm")
-    (fp_text reference SW1 (at 3.25 -2 180) (layer F.SilkS)
+    (fp_text reference SW1 (at 3.175 1.905 180) (layer F.SilkS)
       (effects (font (size 1 1) (thickness 0.15)))
     )
@@
     (descr https://www.omron.com/ecb/products/pdf/en-b3f.pdf)
     (tags "tact sw push 6mm")
-    (fp_text reference SW2 (at 3.25 -2) (layer F.SilkS)
+    (fp_text reference SW2 (at 3.175 1.905) (layer F.SilkS)
       (effects (font (size 1 1) (thickness 0.15)))
     )
@@
     (descr "single turn cermet trimmer, Copal CT-6EP, https://www.nidec-copal-electronics.com/e/catalog/trimmer/ct-6.pdf")
     (tags "potentiometer trimmer")
-    (fp_text reference RV2 (at 0 -2) (layer F.SilkS)
-      (effects (font (size 1 1) (thickness 0.15)))
-    )
-    (fp_text value 10k (at 0 7) (layer F.Fab)
+    (fp_text reference RV2 (at 0 2.54) (layer F.SilkS)
+      (effects (font (size 1 1) (thickness 0.15)))
+    )
+    (fp_text value 10k (at 5.08 3.81) (layer F.SilkS)
       (effects (font (size 1 1) (thickness 0.15)))
     )
@@
       (effects (font (size 1 1) (thickness 0.15)))
     )
-    (fp_text value 680 (at 5.08 2.31 270) (layer F.Fab)
+    (fp_text value 680 (at 5.08 2.31 270) (layer F.SilkS)
       (effects (font (size 1 1) (thickness 0.15)))
     )
@@
     (descr "LED, diameter 3.0mm, 2 pins")
     (tags "LED diameter 3.0mm 2 pins")
-    (fp_text reference D1 (at 1.27 -2.96 90) (layer F.SilkS)
-      (effects (font (size 1 1) (thickness 0.15)))
-    )
-    (fp_text value LED (at 1.27 2.96 90) (layer F.Fab)
+    (fp_text reference D1 (at 1.27 -2.96 90) (layer F.Fab)
+      (effects (font (size 1 1) (thickness 0.15)))
+    )
+    (fp_text value LED (at 1.27 2.96 90) (layer F.SilkS)
       (effects (font (size 1 1) (thickness 0.15)))
     )
@@
       (effects (font (size 1 1) (thickness 0.15)))
     )
-    (fp_text value 4,7µ (at 0.75 3.31 90) (layer F.Fab)
+    (fp_text value 4,7µ (at -2.03 3.29 180) (layer F.SilkS)
       (effects (font (size 1 1) (thickness 0.15)))
     )
@@
     (at 128.905 79.375)
     (descr "2-way 5mm pitch terminal block, Phoenix MKDS series")
-    (fp_text reference J3 (at 2.5 5.9) (layer F.SilkS)
+    (fp_text reference J3 (at 2.54 1.27) (layer F.SilkS)
       (effects (font (size 1 1) (thickness 0.15)))
     )
@@
     (at 139.065 79.375)
     (descr "2-way 5mm pitch terminal block, Phoenix MKDS series")
-    (fp_text reference J2 (at 2.5 5.9) (layer F.SilkS)
+    (fp_text reference J2 (at 2.54 1.27) (layer F.SilkS)
       (effects (font (size 1 1) (thickness 0.15)))
     )
@@
     (at 149.225 79.375)
     (descr "2-way 5mm pitch terminal block, Phoenix MKDS series")
-    (fp_text reference J1 (at 2.5 5.9) (layer F.SilkS)
-      (effects (font (size 1 1) (thickness 0.15)))
-    )
+    (fp_text reference J1 (at 2.54 1.27) (layer F.SilkS)
+      (effects (font (size 1 1) (thickness 0.15)))
+    )

Commit message: correct capacitor
Parts:
- moved C1 1.93 mm to (130.2, 106.0), turned to 270 degrees
Connections:
- C1 pad 1: GND -> 9V
- C1 pad 2: 9V -> GND
Routing:
- net 9V: track 100.4 -> 99.9 mm
