File: Batterietester.kicad_pcb (KiCad board)
At the start: 2 copper layers, 67 x 53 mm, 22 parts, among them J1 Screw_Terminal_1x02, J2 Screw_Terminal_1x02, J3 Screw_Terminal_1x02, J4 CONN_01X02, SW1 SW_Push, SW2 SW_Push, U1 LM3914

Commit message: change open hardware
Parts:
- removed openhardware: OSHW-Logo2_9.8x8mm_SilkScreen, Symbols:OSHW-Logo2_9.8x8mm_SilkScreen
- added LOGO1: OPEN_HARDWARE_1, Symbols:OSHW-Logo2_9.8x8mm_SilkScreen, F.Cu at (132.7, 114.9)
