File: Batterietester.sch (KiCad schematic (older format))
At the start: 15 parts, among them J1 Load, J2 Power, SW1 SW_Push, SW2 SW_Push, U1 LM3914

Commit message: Board design
Parts:
- added J3: Load, Pin_Headers:Pin_Header_Angled_1x02_Pitch2.54mm, symbol CONN_01X02
- J1, J2: footprint Pin_Headers:Pin_Header_Straight_1x02_Pitch2.54mm -> Pin_Headers:Pin_Header_Angled_1x02_Pitch2.54mm
Connections:
- net GND: now also J3.1 (P1)
- net SW_L: now also J3.2 (P2)
Other:
- moved on the sheet: C1, D1, R3, SW2
Changed lines of the file:
@@
 L C C1
 U 1 1 59FF1D94
-P 3750 2350
-F 0 "C1" H 3775 2450 50  0000 L CNN
-F 1 "4,7µ" H 3775 2250 50  0000 L CNN
-F 2 "Capacitors_ThroughHole:CP_Radial_D4.0mm_P1.50mm" H 3788 2200 50  0001 C CNN
-F 3 "" H 3750 2350 50  0001 C CNN
-	1    3750 2350
+P 3300 2350
+F 0 "C1" H 3325 2450 50  0000 L CNN
+F 1 "4,7µ" H 3325 2250 50  0000 L CNN
+F 2 "Capacitors_ThroughHole:CP_Radial_D4.0mm_P1.50mm" H 3338 2200 50  0001 C CNN
+F 3 "" H 3300 2350 50  0001 C CNN
+	1    3300 2350
 	0    1    1    0
 $EndComp
@@
 L GND #PWR01
 U 1 1 59FF1E61
-P 3900 2350
-F 0 "#PWR01" H 3900 2100 50  0001 C CNN
-F 1 "GND" H 3900 2200 50  0000 C CNN
-F 2 "" H 3900 2350 50  0001 C CNN
-F 3 "" H 3900 2350 50  0001 C CNN
-	1    3900 2350
+P 3450 2350
+F 0 "#PWR01" H 3450 2100 50  0001 C CNN
+F 1 "GND" H 3450 2200 50  0000 C CNN
+F 2 "" H 3450 2350 50  0001 C CNN
+F 3 "" H 3450 2350 50  0001 C CNN
+	1    3450 2350
 	0    -1   -1   0
 $EndComp
@@
 L PWR_FLAG #FLG02
 U 1 1 59FF3884
-P 3250 2500
-F 0 "#FLG02" H 3250 2575 50  0001 C CNN
-F 1 "PWR_FLAG" H 3250 2650 50  0000 C CNN
-F 2 "" H 3250 2500 50  0001 C CNN
-F 3 "" H 3250 2500 50  0001 C CNN
-	1    3250 2500
+P 2950 2450
+F 0 "#FLG02" H 2950 2525 50  0001 C CNN
+F 1 "PWR_FLAG" H 2950 2600 50  0000 C CNN
+F 2 "" H 2950 2450 50  0001 C CNN
+F 3 "" H 2950 2450 50  0001 C CNN
+	1    2950 2450
 	-1   0    0    1
 $EndComp
@@
 F 0 "J1" H 1300 4200 50  0000 C CNN
 F 1 "Load" V 1400 4050 50  0000 C CNN
-F 2 "Pin_Headers:Pin_Header_Straight_1x02_Pitch2.54mm" H 1300 4050 50  0001 C CNN
+F 2 "Pin_Headers:Pin_Header_Angled_1x02_Pitch2.54mm" H 1300 4050 50  0001 C CNN
 F 3 "" H 1300 4050 50  0001 C CNN
 	1    1300 4050
@@
 F 0 "J2" H 2100 2550 50  0000 C CNN
 F 1 "Power" V 2200 2400 50  0000 C CNN
-F 2 "Pin_Headers:Pin_Header_Straight_1x02_Pitch2.54mm" H 2100 2400 50  0001 C CNN
+F 2 "Pin_Headers:Pin_Header_Angled_1x02_Pitch2.54mm" H 2100 2400 50  0001 C CNN
 F 3 "" H 2100 2400 50  0001 C CNN
 	1    2100 2400
@@
 	1    0    0    -1
 $EndComp
-Text GLabel 1900 3800 2    60   Input ~ 0
+Text GLabel 2050 3800 1    60   Input ~ 0
 SW_L
 Text GLabel 2150 3300 2    60   Input ~ 0
@@
 L VCC #PWR011
 U 1 1 5A00B84A
-P 3250 1750
-F 0 "#PWR011" H 3250 1600 50  0001 C CNN
-F 1 "VCC" H 3250 1900 50  0000 C CNN
-F 2 "" H 3250 1750 50  0001 C CNN
-F 3 "" H 3250 1750 50  0001 C CNN
-	1    3250 1750
+P 2950 1750
+F 0 "#PWR011" H 2950 1600 50  0001 C CNN
+F 1 "VCC" H 2950 1900 50  0000 C CNN
+F 2 "" H 2950 1750 50  0001 C CNN
+F 3 "" H 2950 1750 50  0001 C CNN
+	1    2950 1750
 	1    0    0    -1
 $EndComp
@@
 L SW_Push SW2
 U 1 1 5A00CBFD
-P 2850 2350
-F 0 "SW2" H 2900 2450 50  0000 L CNN
-F 1 "SW_Push" H 2850 2290 50  0000 C CNN
-F 2 "Buttons_Switches_ThroughHole:SW_PUSH_6mm" H 2850 2550 50  0001 C CNN
-F 3 "" H 2850 2550 50  0001 C CNN
-	1    2850 2350
+P 2550 2350
+F 0 "SW2" H 2600 2450 50  0000 L CNN
+F 1 "SW_Push" H 2550 2290 50  0000 C CNN
+F 2 "Buttons_Switches_ThroughHole:SW_PUSH_6mm" H 2550 2550 50  0001 C CNN
+F 3 "" H 2550 2550 50  0001 C CNN
+	1    2550 2350
 	1    0    0    -1
 $EndComp
@@
 $EndComp
 $Comp
-L GND #PWR013
-U 1 1 5A00D2AD
-P 4200 1900
-F 0 "#PWR013" H 4200 1650 50  0001 C CNN
-F 1 "GND" H 4200 1750 50  0000 C CNN
-F 2 "" H 4200 1900 50  0001 C CNN
-F 3 "" H 4200 1900 50  0001 C CNN
-	1    4200 1900
-	0    -1   -1   0
-$EndComp
-$Comp
 L R R3
 U 1 1 5A00D357
-P 3450 1900
-F 0 "R3" V 3530 1900 50  0000 C CNN
-F 1 "680" V 3450 1900 50  0000 C CNN
-F 2 "Resistors_ThroughHole:R_Axial_DIN0207_L6.3mm_D2.5mm_P10.16mm_Horizontal" V 3380 1900 50  0001 C CNN
-F 3 "" H 3450 1900 50  0001 C CNN
-	1    3450 1900
+P 3300 1900
+F 0 "R3" V 3380 1900 50  0000 C CNN
+F 1 "680" V 3300 1900 50  0000 C CNN
+F 2 "Resistors_ThroughHole:R_Axial_DIN0207_L6.3mm_D2.5mm_P10.16mm_Horizontal" V 3230 1900 50  0001 C CNN
+F 3 "" H 3300 1900 50  0001 C CNN
+	1    3300 1900
 	0    1    1    0
 $EndComp
@@
 L LED D1
 U 1 1 5A00D250
-P 3950 1900
-F 0 "D1" H 3950 2000 50  0000 C CNN
-F 1 "LED" H 3950 1800 50  0000 C CNN
-F 2 "LEDs:LED_D3.0mm" H 3950 1900 50  0001 C CNN
-F 3 "" H 3950 1900 50  0001 C CNN
-	1    3950 1900
-	-1   0    0    1
+P 3600 1900
+F 0 "D1" H 3600 2000 50  0000 C CNN
+F 1 "LED" H 3600 1800 50  0000 C CNN
+F 2 "LEDs:LED_D3.0mm" H 3600 1900 50  0001 C CNN
+F 3 "" H 3600 1900 50  0001 C CNN
+	1    3600 1900
+	-1   0    0    1
+$EndComp
+$Comp
+L GND #PWR013
+U 1 1 5A060BBC
+P 3750 1900
+F 0 "#PWR013" H 3750 1650 50  0001 C CNN
+F 1 "GND" H 3750 1750 50  0000 C CNN
+F 2 "" H 3750 1900 50  0001 C CNN
+F 3 "" H 3750 1900 50  0001 C CNN
+	1    3750 1900
+	0    -1   -1   0
+$EndComp
+$Comp
+L CONN_01X02 J3
+U 1 1 5A06115B
+P 2650 4050
+F 0 "J3" H 2650 4200 50  0000 C CNN
+F 1 "Load" V 2750 4050 50  0000 C CNN
+F 2 "Pin_Headers:Pin_Header_Angled_1x02_Pitch2.54mm" H 2650 4050 50  0001 C CNN
+F 3 "" H 2650 4050 50  0001 C CNN
+	1    2650 4050
+	1    0    0    -1
 $EndComp
 Wire Wire Line
@@
 	6000 1500 6150 1500
 Wire Wire Line
-	1900 3800 1500 3800
-Wire Wire Line
 	1500 4300 1500 4100
-Wire Wire Line
-	1900 4300 1500 4300
 Wire Wire Line
 	1900 4200 1900 4300
@@
 	6500 2200 7350 2200
 Wire Wire Line
-	3050 2350 3600 2350
+	2750 2350 3150 2350
 Connection ~ 10850 3800
 Wire Wire Line
@@
 Connection ~ 2300 2650
 Wire Wire Line
-	2300 2350 2650 2350
-Wire Wire Line
-	4100 1900 4200 1900
-Wire Wire Line
-	3800 1900 3600 1900
-Wire Wire Line
-	3300 1900 3250 1900
-Wire Wire Line
-	3250 1750 3250 2500
-Connection ~ 3250 2350
-Connection ~ 3250 1900
+	2300 2350 2350 2350
+Wire Wire Line
+	3150 1900 2950 1900
+Wire Wire Line
+	2950 1750 2950 2450
+Connection ~ 2950 2350
+Connection ~ 2950 1900
+Connection ~ 1900 4300
+Connection ~ 1900 3800
+Wire Wire Line
+	2450 4100 2250 4100
+Wire Wire Line
+	2250 4100 2250 3800
+Wire Wire Line
+	2250 3800 1500 3800
+Wire Wire Line
+	2450 4300 2450 4000
+Wire Wire Line
+	1500 4300 2450 4300
 $EndSCHEMATC

Commit message: added mounting holes added mode jumper
Parts:
- removed R5: 10k, Resistors_ThroughHole:R_Axial_DIN0207_L6.3mm_D2.5mm_P10.16mm_Horizontal, symbol R
- added J4: CONN_01X02, symbol CONN_01X02
- J1: value Load -> CONN_01X02; footprint Pin_Headers:Pin_Header_Angled_1x02_Pitch2.54mm -> (none)
- J2: value Power -> CONN_01X02; footprint Pin_Headers:Pin_Header_Angled_1x02_Pitch2.54mm -> (none)
- renumbered R3 to R2, R2 to R3
Connections:
- net VCC: now also J4.2 (P2)
- net at U1.9 (Mode): now also J4.1 (P1)
Changed lines of the file:
@@
 $EndDescr
 $Comp
-L R R2
+L R R3
 U 1 1 59FF1797
 P 6150 2500
-F 0 "R2" V 6230 2500 50  0000 C CNN
+F 0 "R3" V 6230 2500 50  0000 C CNN
 F 1 "10k" V 6150 2500 50  0000 C CNN
 F 2 "Resistors_ThroughHole:R_Axial_DIN0207_L6.3mm_D2.5mm_P10.16mm_Horizontal" V 6080 2500 50  0001 C CNN
@@
 L PWR_FLAG #FLG02
 U 1 1 59FF3884
-P 2950 2450
-F 0 "#FLG02" H 2950 2525 50  0001 C CNN
-F 1 "PWR_FLAG" H 2950 2600 50  0000 C CNN
-F 2 "" H 2950 2450 50  0001 C CNN
-F 3 "" H 2950 2450 50  0001 C CNN
-	1    2950 2450
+P 2950 2350
+F 0 "#FLG02" H 2950 2425 50  0001 C CNN
+F 1 "PWR_FLAG" H 2950 2500 50  0000 C CNN
+F 2 "" H 2950 2350 50  0001 C CNN
+F 3 "" H 2950 2350 50  0001 C CNN
+	1    2950 2350
 	-1   0    0    1
 $EndComp
@@
 Obere\nSpannungsgrenze
 $Comp
-L CONN_01X02 J1
-U 1 1 59FF4B69
-P 1300 4050
-F 0 "J1" H 1300 4200 50  0000 C CNN
-F 1 "Load" V 1400 4050 50  0000 C CNN
-F 2 "Pin_Headers:Pin_Header_Angled_1x02_Pitch2.54mm" H 1300 4050 50  0001 C CNN
-F 3 "" H 1300 4050 50  0001 C CNN
-	1    1300 4050
-	-1   0    0    1
-$EndComp
-$Comp
 L R R1
 U 1 1 59FF4C6E
@@
 Text GLabel 5900 1650 0    60   Input ~ 0
 Sig
-$Comp
-L CONN_01X02 J2
-U 1 1 59FF558B
-P 2100 2400
-F 0 "J2" H 2100 2550 50  0000 C CNN
-F 1 "Power" V 2200 2400 50  0000 C CNN
-F 2 "Pin_Headers:Pin_Header_Angled_1x02_Pitch2.54mm" H 2100 2400 50  0001 C CNN
-F 3 "" H 2100 2400 50  0001 C CNN
-	1    2100 2400
-	-1   0    0    1
-$EndComp
 $Comp
 L GND #PWR09
@@
 $EndComp
 $Comp
-L R R5
-U 1 1 5A00BACA
-P 7050 1800
-F 0 "R5" V 7130 1800 50  0000 C CNN
-F 1 "10k" V 7050 1800 50  0000 C CNN
-F 2 "Resistors_ThroughHole:R_Axial_DIN0207_L6.3mm_D2.5mm_P10.16mm_Horizontal" V 6980 1800 50  0001 C CNN
-F 3 "" H 7050 1800 50  0001 C CNN
-	1    7050 1800
-	0    1    1    0
-$EndComp
-$Comp
-L GND #PWR012
-U 1 1 5A00BC5B
-P 6800 1800
-F 0 "#PWR012" H 6800 1550 50  0001 C CNN
-F 1 "GND" H 6800 1650 50  0000 C CNN
-F 2 "" H 6800 1800 50  0001 C CNN
-F 3 "" H 6800 1800 50  0001 C CNN
-	1    6800 1800
-	1    0    0    -1
-$EndComp
-$Comp
 L SW_Push SW1
 U 1 1 5A00CB2A
@@
 $EndComp
 $Comp
-L R R3
+L R R2
 U 1 1 5A00D357
 P 3300 1900
-F 0 "R3" V 3380 1900 50  0000 C CNN
+F 0 "R2" V 3380 1900 50  0000 C CNN
 F 1 "680" V 3300 1900 50  0000 C CNN
 F 2 "Resistors_ThroughHole:R_Axial_DIN0207_L6.3mm_D2.5mm_P10.16mm_Horizontal" V 3230 1900 50  0001 C CNN
@@
 $EndComp
 $Comp
-L GND #PWR013
+L GND #PWR012
 U 1 1 5A060BBC
 P 3750 1900
-F 0 "#PWR013" H 3750 1650 50  0001 C CNN
+F 0 "#PWR012" H 3750 1650 50  0001 C CNN
 F 1 "GND" H 3750 1750 50  0000 C CNN
 F 2 "" H 3750 1900 50  0001 C CNN
@@
 $EndComp
 Wire Wire Line
-	6900 1800 6800 1800
-Wire Wire Line
 	7350 1800 7200 1800
 Wire Wire Line
@@
 	3150 1900 2950 1900
 Wire Wire Line
-	2950 1750 2950 2450
-Connection ~ 2950 2350
+	2950 1750 2950 2350
 Connection ~ 2950 1900
 Connection ~ 1900 4300
@@
 Wire Wire Line
 	1500 4300 2450 4300
+Connection ~ 2950 2350
+$Comp
+L CONN_01X02 J4
+U 1 1 5A07415E
+P 7000 1750
+F 0 "J4" H 7000 1900 50  0000 C CNN
+F 1 "CONN_01X02" V 7100 1750 50  0000 C CNN
+F 2 "" H 7000 1750 50  0001 C CNN
+F 3 "" H 7000 1750 50  0001 C CNN
+	1    7000 1750
+	-1   0    0    1
+$EndComp
+$Comp
+L CONN_01X02 J2
+U 1 1 5A074201
+P 2100 2400
+F 0 "J2" H 2100 2550 50  0000 C CNN
+F 1 "CONN_01X02" V 2200 2400 50  0000 C CNN
+F 2 "" H 2100 2400 50  0001 C CNN
+F 3 "" H 2100 2400 50  0001 C CNN
+	1    2100 2400
+	-1   0    0    1
+$EndComp
+$Comp
+L CONN_01X02 J1
+U 1 1 5A0742F8
+P 1300 4050
+F 0 "J1" H 1300 4200 50  0000 C CNN
+F 1 "CONN_01X02" V 1400 4050 50  0000 C CNN
+F 2 "" H 1300 4050 50  0001 C CNN
+F 3 "" H 1300 4050 50  0001 C CNN
+	1    1300 4050
+	-1   0    0    1
+$EndComp
+Text GLabel 7200 1700 2    60   Input ~ 0
+9V
+Text GLabel 2950 2100 2    60   Input ~ 0
+9V
 $EndSCHEMATC

Commit message: foobar
Parts:
- J1, J2: footprint (none) -> Pin_Headers:Pin_Header_Angled_1x02_Pitch2.54mm
- J3: value Load -> CONN_01X02
- J4: footprint (none) -> Pin_Headers:Pin_Header_Straight_1x02_Pitch2.54mm
Changed lines of the file:
@@
 	0    -1   -1   0
-$EndComp
-$Comp
-L CONN_01X02 J3
-U 1 1 5A06115B
-P 2650 4050
-F 0 "J3" H 2650 4200 50  0000 C CNN
-F 1 "Load" V 2750 4050 50  0000 C CNN
-F 2 "Pin_Headers:Pin_Header_Angled_1x02_Pitch2.54mm" H 2650 4050 50  0001 C CNN
-F 3 "" H 2650 4050 50  0001 C CNN
-	1    2650 4050
-	1    0    0    -1
 $EndComp
 Wire Wire Line
@@
 F 0 "J4" H 7000 1900 50  0000 C CNN
 F 1 "CONN_01X02" V 7100 1750 50  0000 C CNN
-F 2 "" H 7000 1750 50  0001 C CNN
+F 2 "Pin_Headers:Pin_Header_Straight_1x02_Pitch2.54mm" H 7000 1750 50  0001 C CNN
 F 3 "" H 7000 1750 50  0001 C CNN
 	1    7000 1750
@@
 F 0 "J2" H 2100 2550 50  0000 C CNN
 F 1 "CONN_01X02" V 2200 2400 50  0000 C CNN
-F 2 "" H 2100 2400 50  0001 C CNN
+F 2 "Pin_Headers:Pin_Header_Angled_1x02_Pitch2.54mm" H 2100 2400 50  0001 C CNN
 F 3 "" H 2100 2400 50  0001 C CNN
 	1    2100 2400
@@
 F 0 "J1" H 1300 4200 50  0000 C CNN
 F 1 "CONN_01X02" V 1400 4050 50  0000 C CNN
-F 2 "" H 1300 4050 50  0001 C CNN
+F 2 "Pin_Headers:Pin_Header_Angled_1x02_Pitch2.54mm" H 1300 4050 50  0001 C CNN
 F 3 "" H 1300 4050 50  0001 C CNN
 	1    1300 4050
@@
 Text GLabel 2950 2100 2    60   Input ~ 0
 9V
+$Comp
+L CONN_01X02 J3
+U 1 1 5A0749A6
+P 2650 4050
+F 0 "J3" H 2650 4200 50  0000 C CNN
+F 1 "CONN_01X02" V 2750 4050 50  0000 C CNN
+F 2 "Pin_Headers:Pin_Header_Angled_1x02_Pitch2.54mm" H 2650 4050 50  0001 C CNN
+F 3 "" H 2650 4050 50  0001 C CNN
+	1    2650 4050
+	1    0    0    -1
+$EndComp
 $EndSCHEMATC
