File: Batterietester.sch (KiCad schematic (older format))
At the start: 16 parts, among them J1 Screw_Terminal_1x02, J2 Screw_Terminal_1x02, J3 Screw_Terminal_1x02, J4 CONN_01X02, SW1 SW_Push, SW2 SW_Push, U1 LM3914

Commit message: change open hardware
Parts:
- added LOGO1: OPEN_HARDWARE_1, Symbols:OSHW-Logo2_9.8x8mm_SilkScreen, symbol OPEN_HARDWARE_1
Changed lines of the file:
@@
 	0    -1   -1   0
 $EndComp
+$Comp
+L OPEN_HARDWARE_1 LOGO1
+U 1 1 5A22E89B
+P 10400 5950
+F 0 "LOGO1" H 10400 6225 50  0000 C CNN
+F 1 "OPEN_HARDWARE_1" H 10400 5725 50  0000 C CNN
+F 2 "Symbols:OSHW-Logo2_9.8x8mm_SilkScreen" H 10400 5950 50  0001 C CNN
+F 3 "" H 10400 5950 50  0001 C CNN
+	1    10400 5950
+	1    0    0    -1
+$EndComp
 $EndSCHEMATC
